Commit message: working ns moveit

File: urdf/ur5_gazebo.xacro (robot description, xacro)
@@ -4,5 +4,5 @@
 <xacro:arg name="robot_namespace" default="" />
 <xacro:property name="robot_namespace" value="$(arg robot_namespace)" />
-<xacro:property name="ns_prefix" value="${robot_namespace + '_' if robot_namespace else ''}" />
+<xacro:property name="ns_prefix" value="" />
 <xacro:property name="body_color" value="Gazebo/Silver" />
 <xacro:property name="p_gain" value="10"/>

File: urdf/ur5_ros2_control.xacro (robot description, xacro)
@@ -4,5 +4,5 @@
     <xacro:arg name="robot_namespace" default="" />
     <xacro:property name="robot_namespace" value="$(arg robot_namespace)" />
-    <xacro:property name="ns_prefix" value="${robot_namespace + '_' if robot_namespace else ''}" />
+    <xacro:property name="ns_prefix" value="" />
     <ros2_control name="GazeboSystem" type="system">
         <hardware>
