Commit message: temporary fix

File: urdf/mobile_manipulator.urdf.xacro (robot description, xacro)
@@ -51,5 +51,5 @@
   <!-- We need to define the UR5 arm structure inline or include it with proper parent -->
   <!-- UR5 Base Link mounted on the arm mounting plate -->
-  <link name="${ns_prefix}ur5_base_link">
+  <link name="${ns_prefix}arm_base_link">
     <inertial>
       <origin xyz="-0.0033230512143046006 -0.0004232197888539764 0.037822190938846395" rpy="0 0 0"/>
@@ -79,11 +79,11 @@
   </link>
   <!-- Joint connecting UR5 base to the mounting plate -->
-  <joint name="${ns_prefix}ur5_mount_joint" type="fixed">
+  <joint name="${ns_prefix}arm_mount_base_joint" type="fixed">
     <parent link="${ns_prefix}arm_mount_plate"/>
-    <child link="${ns_prefix}ur5_base_link"/>
+    <child link="${ns_prefix}arm_base_link"/>
     <origin xyz="0 0 -0.025" rpy="0 0 0"/>
   </joint>
   <!-- UR5 Link 1 -->
-  <link name="${ns_prefix}ur5_link1_1">
+  <link name="${ns_prefix}arm_link1_1">
     <inertial>
       <origin xyz="-5.118812714607554e-06 0.016411047782836283 0.05864433019110279" rpy="0 0 0"/>
@@ -105,12 +105,12 @@
     </collision>
   </link>
-  <joint name="${ns_prefix}ur5_base_link1_joint" type="continuous">
+  <joint name="${ns_prefix}arm_base_link1_joint" type="continuous">
     <origin xyz="-0.003691 -5.6e-05 0.050586" rpy="0 0 0"/>
-    <parent link="${ns_prefix}ur5_base_link"/>
-    <child link="${ns_prefix}ur5_link1_1"/>
+    <parent link="${ns_prefix}arm_base_link"/>
+    <child link="${ns_prefix}arm_link1_1"/>
     <axis xyz="0.0 -0.0 1.0"/>
   </joint>
   <!-- UR5 Link 2 Part 1 -->
-  <link name="${ns_prefix}ur5_link2_p1_1">
+  <link name="${ns_prefix}arm_link2_p1_1">
     <inertial>
       <origin xyz="6.203040415705269e-06 0.06207005674361077 0.007860389181770538" rpy="0 0 0"/>
@@ -132,12 +132,12 @@
     </collision>
   </link>
-  <joint name="${ns_prefix}ur5_link1_link2p1_joint" type="continuous">
+  <joint name="${ns_prefix}arm_link1_link2p1_joint" type="continuous">
     <origin xyz="0.0 0.0753 0.0597" rpy="0 0 0"/>
-    <parent link="${ns_prefix}ur5_link1_1"/>
-    <child link="${ns_prefix}ur5_link2_p1_1"/>
+    <parent link="${ns_prefix}arm_link1_1"/>
+    <child link="${ns_prefix}arm_link2_p1_1"/>
     <axis xyz="0.0 -1.0 -0.0"/>
   </joint>
   <!-- UR5 Link 2 Part 2 -->
-  <link name="${ns_prefix}ur5_link2_p2_1">
+  <link name="${ns_prefix}arm_link2_p2_1">
     <inertial>
       <origin xyz="-8.752471172565526e-05 2.4376620175181607e-07 0.1524996678439083" rpy="0 0 0"/>
@@ -159,11 +159,11 @@
     </collision>
   </link>
-  <joint name="${ns_prefix}ur5_p1_p2_joint" type="fixed">
+  <joint name="${ns_prefix}arm_p1_p2_joint" type="fixed">
     <origin xyz="-2e-06 0.067003 0.0663" rpy="0 0 0"/>
-    <parent link="${ns_prefix}ur5_link2_p1_1"/>
-    <child link="${ns_prefix}ur5_link2_p2_1"/>
+    <parent link="${ns_prefix}arm_link2_p1_1"/>
+    <child link="${ns_prefix}arm_link2_p2_1"/>
   </joint>
   <!-- UR5 Link 2 Part 3 -->
-  <link name="${ns_prefix}ur5_link2_p3_1">
+  <link name="${ns_prefix}arm_link2_p3_1">
     <inertial>
       <origin xyz="-7.763250047288905e-06 -0.004932943256389266 0.05843895228729162" rpy="0 0 0"/>
@@ -185,11 +185,11 @@
     </collision>
   </link>
-  <joint name="${ns_prefix}ur5_p2_p3_joint" type="fixed">
+  <joint name="${ns_prefix}arm_p2_p3_joint" type="fixed">
     <origin xyz="-1.1e-05 0.0 0.305" rpy="0 0 0"/>
-    <parent link="${ns_prefix}ur5_link2_p2_1"/>
-    <child link="${ns_prefix}ur5_link2_p3_1"/>
+    <parent link="${ns_prefix}arm_link2_p2_1"/>
+    <child link="${ns_prefix}arm_link2_p3_1"/>
   </joint>
   <!-- UR5 Link 3 -->
-  <link name="${ns_prefix}ur5_link3_1">
+  <link name="${ns_prefix}arm_link3_1">
     <inertial>
       <origin xyz="0.17378102072172863 -0.04787490591742441 0.00100186606907815" rpy="0 0 0"/>
@@ -211,12 +211,12 @@
     </collision>
   </link>
-  <joint name="${ns_prefix}ur5_link2p3_link3_joint" type="continuous">
+  <joint name="${ns_prefix}arm_link2p3_link3_joint" type="continuous">
     <origin xyz="-2e-06 -0.067003 0.0663" rpy="0 0 0"/>
-    <parent link="${ns_prefix}ur5_link2_p3_1"/>
-    <child link="${ns_prefix}ur5_link3_1"/>
+    <parent link="${ns_prefix}arm_link2_p3_1"/>
+    <child link="${ns_prefix}arm_link3_1"/>
     <axis xyz="0.0 -1.0 -0.0"/>
   </joint>
   <!-- UR5 Link 4 -->
-  <link name="${ns_prefix}ur5_link4_1">
+  <link name="${ns_prefix}arm_link4_1">
     <inertial>
       <origin xyz="2.12490884528016e-05 0.04182917130330904 -0.003987177325129543" rpy="0 0 0"/>
@@ -238,12 +238,12 @@
     </collision>
   </link>
-  <joint name="${ns_prefix}ur5_link3_link4_joint" type="continuous">
+  <joint name="${ns_prefix}arm_link3_link4_joint" type="continuous">
     <origin xyz="0.392244 -0.012 0.002256" rpy="0 0 0"/>
-    <parent link="${ns_prefix}ur5_link3_1"/>
-    <child link="${ns_prefix}ur5_link4_1"/>
+    <parent link="${ns_prefix}arm_link3_1"/>
+    <child link="${ns_prefix}arm_link4_1"/>
     <axis xyz="0.0 1.0 -0.0"/>
   </joint>
   <!-- UR5 Link 5 -->
-  <link name="${ns_prefix}ur5_link5_1">
+  <link name="${ns_prefix}arm_link5_1">
     <inertial>
       <origin xyz="-0.003851364362202292 4.3924354040825175e-05 0.04240877360333983" rpy="0 0 0"/>
@@ -265,12 +265,12 @@
     </collision>
   </link>
-  <joint name="${ns_prefix}ur5_link4_link5_joint" type="continuous">
+  <joint name="${ns_prefix}arm_link4_link5_joint" type="continuous">
     <origin xyz="-9.7e-05 0.05362 0.04155" rpy="0 0 0"/>
-    <parent link="${ns_prefix}ur5_link4_1"/>
-    <child link="${ns_prefix}ur5_link5_1"/>
+    <parent link="${ns_prefix}arm_link4_1"/>
+    <child link="${ns_prefix}arm_link5_1"/>
     <axis xyz="-0.00232 0.0 0.999997"/>
   </joint>
   <!-- UR5 Link 6 -->
-  <link name="${ns_prefix}ur5_link6_1">
+  <link name="${ns_prefix}arm_link6_1">
     <inertial>
       <origin xyz="0.01818377138506838 -7.537991570427671e-05 0.0001621667781095404" rpy="0 0 0"/>
@@ -292,12 +292,12 @@
     </collision>
   </link>
-  <joint name="${ns_prefix}ur5_link5_link6_joint" type="continuous">
+  <joint name="${ns_prefix}arm_link5_link6_joint" type="continuous">
     <origin xyz="0.041424 -0.000352 0.053716" rpy="0 0 0"/>
-    <parent link="${ns_prefix}ur5_link5_1"/>
-    <child link="${ns_prefix}ur5_link6_1"/>
+    <parent link="${ns_prefix}arm_link5_1"/>
+    <child link="${ns_prefix}arm_link6_1"/>
     <axis xyz="0.999962 -0.008461 0.00232"/>
   </joint>
   <!-- Gazebo tags for UR5 links -->
-  <gazebo reference="${ns_prefix}ur5_base_link">
+  <gazebo reference="${ns_prefix}arm_base_link">
     <material>Gazebo/Silver</material>
     <mu1>0.2</mu1>
@@ -306,47 +306,47 @@
     <gravity>true</gravity>
   </gazebo>
-  <gazebo reference="${ns_prefix}ur5_link1_1">
-    <material>Gazebo/Silver</material>
-    <mu1>0.2</mu1>
-    <mu2>0.2</mu2>
-    <self_collide>true</self_collide>
-  </gazebo>
-  <gazebo reference="${ns_prefix}ur5_link2_p1_1">
-    <material>Gazebo/Silver</material>
-    <mu1>0.2</mu1>
-    <mu2>0.2</mu2>
-    <self_collide>true</self_collide>
-  </gazebo>
-  <gazebo reference="${ns_prefix}ur5_link2_p2_1">
-    <material>Gazebo/Silver</material>
-    <mu1>0.2</mu1>
-    <mu2>0.2</mu2>
-    <self_collide>true</self_collide>
-  </gazebo>
-  <gazebo reference="${ns_prefix}ur5_link2_p3_1">
-    <material>Gazebo/Silver</material>
-    <mu1>0.2</mu1>
-    <mu2>0.2</mu2>
-    <self_collide>true</self_collide>
-  </gazebo>
-  <gazebo reference="${ns_prefix}ur5_link3_1">
-    <material>Gazebo/Silver</material>
-    <mu1>0.2</mu1>
-    <mu2>0.2</mu2>
-    <self_collide>true</self_collide>
-  </gazebo>
-  <gazebo reference="${ns_prefix}ur5_link4_1">
-    <material>Gazebo/Silver</material>
-    <mu1>0.2</mu1>
-    <mu2>0.2</mu2>
-    <self_collide>true</self_collide>
-  </gazebo>
-  <gazebo reference="${ns_prefix}ur5_link5_1">
-    <material>Gazebo/Silver</material>
-    <mu1>0.2</mu1>
-    <mu2>0.2</mu2>
-    <self_collide>true</self_collide>
-  </gazebo>
-  <gazebo reference="${ns_prefix}ur5_link6_1">
+  <gazebo reference="${ns_prefix}arm_link1_1">
+    <material>Gazebo/Silver</material>
+    <mu1>0.2</mu1>
+    <mu2>0.2</mu2>
+    <self_collide>true</self_collide>
+  </gazebo>
+  <gazebo reference="${ns_prefix}arm_link2_p1_1">
+    <material>Gazebo/Silver</material>
+    <mu1>0.2</mu1>
+    <mu2>0.2</mu2>
+    <self_collide>true</self_collide>
+  </gazebo>
+  <gazebo reference="${ns_prefix}arm_link2_p2_1">
+    <material>Gazebo/Silver</material>
+    <mu1>0.2</mu1>
+    <mu2>0.2</mu2>
+    <self_collide>true</self_collide>
+  </gazebo>
+  <gazebo reference="${ns_prefix}arm_link2_p3_1">
+    <material>Gazebo/Silver</material>
+    <mu1>0.2</mu1>
+    <mu2>0.2</mu2>
+    <self_collide>true</self_collide>
+  </gazebo>
+  <gazebo reference="${ns_prefix}arm_link3_1">
+    <material>Gazebo/Silver</material>
+    <mu1>0.2</mu1>
+    <mu2>0.2</mu2>
+    <self_collide>true</self_collide>
+  </gazebo>
+  <gazebo reference="${ns_prefix}arm_link4_1">
+    <material>Gazebo/Silver</material>
+    <mu1>0.2</mu1>
+    <mu2>0.2</mu2>
+    <self_collide>true</self_collide>
+  </gazebo>
+  <gazebo reference="${ns_prefix}arm_link5_1">
+    <material>Gazebo/Silver</material>
+    <mu1>0.2</mu1>
+    <mu2>0.2</mu2>
+    <self_collide>true</self_collide>
+  </gazebo>
+  <gazebo reference="${ns_prefix}arm_link6_1">
     <material>Gazebo/Silver</material>
     <mu1>0.2</mu1>
@@ -381,45 +381,45 @@
     </joint>
     <!-- UR5 Arm Joints -->
-    <joint name="${ns_prefix}ur5_base_link1_joint">
-      <command_interface name="position">
-        <param name="min">-6.28</param>
-        <param name="max">6.28</param>
-      </command_interface>
-      <state_interface name="position"/>
-      <state_interface name="velocity"/>
-    </joint>
-    <joint name="${ns_prefix}ur5_link1_link2p1_joint">
-      <command_interface name="position">
-        <param name="min">-6.28</param>
-        <param name="max">6.28</param>
-      </command_interface>
-      <state_interface name="position"/>
-      <state_interface name="velocity"/>
-    </joint>
-    <joint name="${ns_prefix}ur5_link2p3_link3_joint">
-      <command_interface name="position">
-        <param name="min">-6.28</param>
-        <param name="max">6.28</param>
-      </command_interface>
-      <state_interface name="position"/>
-      <state_interface name="velocity"/>
-    </joint>
-    <joint name="${ns_prefix}ur5_link3_link4_joint">
-      <command_interface name="position">
-        <param name="min">-6.28</param>
-        <param name="max">6.28</param>
-      </command_interface>
-      <state_interface name="position"/>
-      <state_interface name="velocity"/>
-    </joint>
-    <joint name="${ns_prefix}ur5_link4_link5_joint">
-      <command_interface name="position">
-        <param name="min">-6.28</param>
-        <param name="max">6.28</param>
-      </command_interface>
-      <state_interface name="position"/>
-      <state_interface name="velocity"/>
-    </joint>
-    <joint name="${ns_prefix}ur5_link5_link6_joint">
+    <joint name="${ns_prefix}arm_base_link1_joint">
+      <command_interface name="position">
+        <param name="min">-6.28</param>
+        <param name="max">6.28</param>
+      </command_interface>
+      <state_interface name="position"/>
+      <state_interface name="velocity"/>
+    </joint>
+    <joint name="${ns_prefix}arm_link1_link2p1_joint">
+      <command_interface name="position">
+        <param name="min">-6.28</param>
+        <param name="max">6.28</param>
+      </command_interface>
+      <state_interface name="position"/>
+      <state_interface name="velocity"/>
+    </joint>
+    <joint name="${ns_prefix}arm_link2p3_link3_joint">
+      <command_interface name="position">
+        <param name="min">-6.28</param>
+        <param name="max">6.28</param>
+      </command_interface>
+      <state_interface name="position"/>
+      <state_interface name="velocity"/>
+    </joint>
+    <joint name="${ns_prefix}arm_link3_link4_joint">
+      <command_interface name="position">
+        <param name="min">-6.28</param>
+        <param name="max">6.28</param>
+      </command_interface>
+      <state_interface name="position"/>
+      <state_interface name="velocity"/>
+    </joint>
+    <joint name="${ns_prefix}arm_link4_link5_joint">
+      <command_interface name="position">
+        <param name="min">-6.28</param>
+        <param name="max">6.28</param>
+      </command_interface>
+      <state_interface name="position"/>
+      <state_interface name="velocity"/>
+    </joint>
+    <joint name="${ns_prefix}arm_link5_link6_joint">
       <command_interface name="position">
         <param name="min">-6.28</param>
