Commit message: server migration v1

File: urdf/detachable_joints.xacro (robot description, xacro)
@@ -28,5 +28,5 @@
   <!-- NOTE: Boxes 24 and 25 are EXCLUDED because they don't exist in the world -->
   <xacro:macro name="detachable_joints_all_boxes" params="parent_link robot_ns">
-    <!-- Boxes 0-23 -->
+    <!-- Boxes 0-23 (COMMENTED OUT - not spawned in current simulation)
     <xacro:detachable_joint_for_box parent_link="${parent_link}" box_id="0" robot_ns="${robot_ns}"/>
     <xacro:detachable_joint_for_box parent_link="${parent_link}" box_id="1" robot_ns="${robot_ns}"/>
@@ -53,6 +53,7 @@
     <xacro:detachable_joint_for_box parent_link="${parent_link}" box_id="22" robot_ns="${robot_ns}"/>
     <xacro:detachable_joint_for_box parent_link="${parent_link}" box_id="23" robot_ns="${robot_ns}"/>
+    -->
     <!-- Boxes 24 and 25 are SKIPPED - they don't exist in the world file -->
-    <!-- Boxes 26-49 -->
+    <!-- Boxes 26-33 (ACTIVE - spawned in current simulation) -->
     <xacro:detachable_joint_for_box parent_link="${parent_link}" box_id="26" robot_ns="${robot_ns}"/>
     <xacro:detachable_joint_for_box parent_link="${parent_link}" box_id="27" robot_ns="${robot_ns}"/>
@@ -63,4 +64,5 @@
     <xacro:detachable_joint_for_box parent_link="${parent_link}" box_id="32" robot_ns="${robot_ns}"/>
     <xacro:detachable_joint_for_box parent_link="${parent_link}" box_id="33" robot_ns="${robot_ns}"/>
+    <!-- Boxes 34-49 (COMMENTED OUT - not spawned in current simulation)
     <xacro:detachable_joint_for_box parent_link="${parent_link}" box_id="34" robot_ns="${robot_ns}"/>
     <xacro:detachable_joint_for_box parent_link="${parent_link}" box_id="35" robot_ns="${robot_ns}"/>
@@ -79,4 +81,5 @@
     <xacro:detachable_joint_for_box parent_link="${parent_link}" box_id="48" robot_ns="${robot_ns}"/>
     <xacro:detachable_joint_for_box parent_link="${parent_link}" box_id="49" robot_ns="${robot_ns}"/>
+    -->
   </xacro:macro>
 </robot>

File: urdf/jackal.urdf.xacro (robot description, xacro)
@@ -221,15 +221,3 @@
     <xacro:include filename="$(find swarm_description)/urdf/jackal_ros2_control.xacro" />
   </xacro:if>
-  <!-- Optional standard accessories, including their simulation data. The rendering
-       of these into the final description is controlled by optenv variables, which
-       default each one to off.-->
-  <xacro:include filename="$(find swarm_description)/urdf/jackal_accessories.urdf.xacro" />
-  <!-- OutdoorNav -->
-  <xacro:arg name="outdoornav_enabled"       default="$(optenv OUTDOORNAV_ENABLED 0)" />
-  <xacro:arg name="outdoornav_configuration" default="$(optenv OUTDOORNAV_CONFIGURATION standard)" />
-  <!-- OutdoorNav URDF Config -->
-  <xacro:if value="$(arg outdoornav_enabled)">
-    <xacro:include filename="$(find cpr_onav_description)/urdf/outdoornav_description.urdf.xacro" />
-    <xacro:outdoornav_sensors outdoornav_configuration="$(arg outdoornav_configuration)" />
-  </xacro:if>
 </robot>

File: urdf/mobile_manipulator.urdf.xacro (robot description, xacro)
@@ -55,11 +55,11 @@
   <link name="${ns_prefix}arm_base_link">
     <inertial>
-      <origin xyz="-0.0033230512143046006 -0.0004232197888539764 0.037822190938846395" rpy="0 0 0"/>
-      <mass value="25.3"/>
+      <origin xyz="0.0 0.0 0.0" rpy="0 0 0"/>
+      <mass value="4.0"/>
       <inertia
-          ixx="0.00671"
-          iyy="0.00671"
-          izz="0.01125"
-          ixy="-0.000188"
+          ixx="0.00443333"
+          iyy="0.00443333"
+          izz="0.0072"
+          ixy="0.0"
           iyz="0.0"
           ixz="0.0"
@@ -89,7 +89,7 @@
   <link name="${ns_prefix}arm_link1_1">
     <inertial>
-      <origin xyz="-5.118812714607554e-06 0.016411047782836283 0.05864433019110279" rpy="0 0 0"/>
-      <mass value="1.667428920912541"/>
-      <inertia ixx="0.004178" iyy="0.003273" izz="0.003817" ixy="0.0" iyz="-0.000173" ixz="1e-06"/>
+      <origin xyz="0.0 -0.02561 0.00193" rpy="0 0 0"/>
+      <mass value="3.7"/>
+      <inertia ixx="0.010267" iyy="0.010267" izz="0.00666" ixy="0.0" iyz="0.0" ixz="0.0"/>
     </inertial>
     <visual>
@@ -116,7 +116,7 @@
   <link name="${ns_prefix}arm_link2_p1_1">
     <inertial>
-      <origin xyz="6.203040415705269e-06 0.06207005674361077 0.007860389181770538" rpy="0 0 0"/>
-      <mass value="1.5524700894200791"/>
-      <inertia ixx="0.003628" iyy="0.003009" izz="0.003383" ixy="-1e-06" iyz="-0.000207" ixz="-0.0"/>
+      <origin xyz="0.0 0.0 0.0" rpy="0 0 0"/>
+      <mass value="2.578"/>
+      <inertia ixx="0.006015" iyy="0.004988" izz="0.005608" ixy="0.0" iyz="0.0" ixz="0.0"/>
     </inertial>
     <visual>
@@ -143,7 +143,7 @@
   <link name="${ns_prefix}arm_link2_p2_1">
     <inertial>
-      <origin xyz="-8.752471172565526e-05 2.4376620175181607e-07 0.1524996678439083" rpy="0 0 0"/>
-      <mass value="1.937681145922208"/>
-      <inertia ixx="0.017402" iyy="0.017402" izz="0.001914" ixy="0.0" iyz="-0.0" ixz="1e-06"/>
+      <origin xyz="0.2125 0.0 0.11336" rpy="0 0 0"/>
+      <mass value="3.237"/>
+      <inertia ixx="0.084669" iyy="0.084669" izz="0.005827" ixy="0.0" iyz="0.0" ixz="0.0"/>
     </inertial>
     <visual>
@@ -169,7 +169,7 @@
   <link name="${ns_prefix}arm_link2_p3_1">
     <inertial>
-      <origin xyz="-7.763250047288905e-06 -0.004932943256389266 0.05843895228729162" rpy="0 0 0"/>
-      <mass value="1.5524700894200791"/>
-      <inertia ixx="0.003628" iyy="0.003009" izz="0.003383" ixy="1e-06" iyz="0.000207" ixz="-0.0"/>
+      <origin xyz="0.0 0.0 0.0" rpy="0 0 0"/>
+      <mass value="2.578"/>
+      <inertia ixx="0.006015" iyy="0.004988" izz="0.005608" ixy="0.0" iyz="0.0" ixz="0.0"/>
     </inertial>
     <visual>
@@ -195,7 +195,7 @@
   <link name="${ns_prefix}arm_link3_1">
     <inertial>
-      <origin xyz="0.17378102072172863 -0.04787490591742441 0.00100186606907815" rpy="0 0 0"/>
-      <mass value="2.846539405621545"/>
-      <inertia ixx="0.003063" iyy="0.061797" izz="0.062318" ixy="0.003731" iyz="2.2e-05" ixz="-0.000342"/>
+      <origin xyz="0.11993 0.0 0.0265" rpy="0 0 0"/>
+      <mass value="2.275"/>
+      <inertia ixx="0.004095" iyy="0.004095" izz="0.002049" ixy="0.0" iyz="0.0" ixz="0.0"/>
     </inertial>
     <visual>
@@ -222,7 +222,7 @@
   <link name="${ns_prefix}arm_link4_1">
     <inertial>
-      <origin xyz="2.12490884528016e-05 0.04182917130330904 -0.003987177325129543" rpy="0 0 0"/>
-      <mass value="0.5732810659722621"/>
-      <inertia ixx="0.000753" iyy="0.000581" izz="0.000587" ixy="0.0" iyz="1.1e-05" ixz="0.0"/>
+      <origin xyz="0.0 -0.0018 0.01634" rpy="0 0 0"/>
+      <mass value="1.219"/>
+      <inertia ixx="0.002110" iyy="0.002110" izz="0.002194" ixy="0.0" iyz="0.0" ixz="0.0"/>
     </inertial>
     <visual>
@@ -249,7 +249,7 @@
   <link name="${ns_prefix}arm_link5_1">
     <inertial>
-      <origin xyz="-0.003851364362202292 4.3924354040825175e-05 0.04240877360333983" rpy="0 0 0"/>
-      <mass value="0.5732811937839646"/>
-      <inertia ixx="0.000597" iyy="0.000754" izz="0.000572" ixy="1e-06" iyz="0.0" ixz="2e-05"/>
+      <origin xyz="0.0 0.0018 0.01634" rpy="0 0 0"/>
+      <mass value="1.219"/>
+      <inertia ixx="0.002110" iyy="0.002110" izz="0.002194" ixy="0.0" iyz="0.0" ixz="0.0"/>
     </inertial>
     <visual>
@@ -276,7 +276,7 @@
   <link name="${ns_prefix}arm_link6_1">
     <inertial>
-      <origin xyz="0.01818377138506838 -7.537991570427671e-05 0.0001621667781095404" rpy="0 0 0"/>
-      <mass value="0.1747134109193075"/>
-      <inertia ixx="0.000123" iyy="8.2e-05" izz="8.3e-05" ixy="-0.0" iyz="0.0" ixz="-0.0"/>
+      <origin xyz="0.0 0.001159 0.0" rpy="0 0 0"/>
+      <mass value="0.1879"/>
+      <inertia ixx="0.000132" iyy="0.000132" izz="0.000101" ixy="0.0" iyz="0.0" ixz="0.0"/>
     </inertial>
     <visual>
@@ -432,5 +432,16 @@
     </joint>
   </ros2_control>
+  <!-- Gazebo ROS2 Control Plugin for Mobile Manipulator -->
+  <gazebo>
+    <plugin name="gz_ros2_control::GazeboSimROS2ControlPlugin" filename="gz_ros2_control-system">
+        <parameters>$(find swarm_description)/config/mobman_control.yaml</parameters>
+        <ros>
+          <namespace>${robot_namespace}</namespace>
+          <remapping>diff_drive_controller/cmd_vel_unstamped:=cmd_vel</remapping>
+          <remapping>diff_drive_controller/odom:=odom</remapping>
+        </ros>
+    </plugin>
+  </gazebo>
   <!-- DetachableJoint plugins for all 48 aruco boxes -->
-  <xacro:detachable_joints_all_boxes parent_link="${ns_prefix}arm_link6_1" robot_ns="mobile_manipulator"/>
+  <xacro:detachable_joints_all_boxes parent_link="${ns_prefix}arm_link6_1" robot_ns="${robot_namespace}"/>
 </robot>

File: urdf/ur5_assembly.xacro (robot description, xacro)
@@ -7,5 +7,4 @@
 <xacro:property name="ns_prefix" value="" />
 <xacro:include filename="$(find swarm_description)/urdf/materials.xacro" />
-<!--<xacro:include filename="$(find swarm_description)/urdf/ur5_assembly.trans" />-->
 <xacro:include filename="$(find swarm_description)/urdf/ur5_gazebo.xacro" />
 <xacro:include filename="$(find swarm_description)/urdf/ur5_ros2_control.xacro" />
@@ -324,4 +323,11 @@
   <child link="${ns_prefix}depth_frame"/>
 </joint>
+<link name="${ns_prefix}optical_frame">
+</link>
+<joint name="${ns_prefix}camera_optical_joint" type="fixed">
+  <origin xyz="0 0 0" rpy="-1.57 0 -1.57"/>
+  <parent link="${ns_prefix}depth_frame"/>
+  <child link="${ns_prefix}optical_frame"/>
+</joint>
 <gazebo reference="${ns_prefix}depth_frame">
   <sensor name="rgbd_camera" type="rgbd_camera">
@@ -331,8 +337,8 @@
       <lens>
         <intrinsics>
-          <fx>277.1</fx>
-          <fy>277.1</fy>
-          <cx>160.5</cx>
-          <cy>120.5</cy>
+          <fx>762.7</fx>
+          <fy>762.7</fy>
+          <cx>640.0</cx>
+          <cy>360.0</cy>
           <s>0</s>
         </intrinsics>
