Commit message: checking the changes

File: urdf/jackal.urdf.xacro (robot description, xacro)
@@ -5,5 +5,5 @@
   <xacro:property name="robot_namespace" value="$(arg robot_namespace)" />
   <!-- Add underscore separator if namespace is not empty -->
-  <xacro:property name="ns_prefix" value="${robot_namespace + '_' if robot_namespace else ''}" />
+  <xacro:property name="ns_prefix" value="" />
   <xacro:property name="PI" value="3.1415926535897931" />
   <xacro:property name="wheelbase" value="0.262" />

File: urdf/jackal_ros2_control.xacro (robot description, xacro)
@@ -4,5 +4,5 @@
     <xacro:arg name="robot_namespace" default="" />
     <xacro:property name="robot_namespace" value="$(arg robot_namespace)" />
-    <xacro:property name="ns_prefix" value="${robot_namespace + '_' if robot_namespace else ''}" />
+    <xacro:property name="ns_prefix" value="" />
     <ros2_control name='JackalController' type='system'>
         <!--

File: urdf/mobile_manipulator.urdf.xacro (robot description, xacro)
@@ -5,5 +5,5 @@
   <xacro:property name="robot_namespace" value="$(arg robot_namespace)" />
   <!-- Add underscore separator if namespace is not empty -->
-  <xacro:property name="ns_prefix" value="${robot_namespace + '_' if robot_namespace else ''}" />
+  <xacro:property name="ns_prefix" value="" />
   <!-- Tell jackal.urdf.xacro not to include its own ros2_control -->
   <xacro:arg name="standalone" default="false" />

Commit message: acomododated atomic pick and place actions

File: urdf/jackal.urdf.xacro (robot description, xacro)
@@ -194,5 +194,5 @@
     <parent link="${ns_prefix}chassis_link" />
     <child link="${ns_prefix}lidar_link" />
-    <origin xyz="0.0 0.0 0.205" />
+    <origin xyz="0.0 0.0 0.1" />
   </joint>
   <link name="${ns_prefix}mid_mount"></link>

File: urdf/mobile_manipulator.urdf.xacro (robot description, xacro)
@@ -36,10 +36,10 @@
     </collision>
     <inertial>
-      <mass value="2.0"/>
+      <mass value="5.0"/>  <!-- Increased from 2.0 to anchor weight at base -->
       <origin xyz="0 0 ${-arm_mount_height/2}" rpy="0 0 0"/>
       <inertia
-        ixx="0.00875" ixy="0.0" ixz="0.0"
-        iyy="0.00875" iyz="0.0"
-        izz="0.015"/>
+        ixx="0.02188" ixy="0.0" ixz="0.0"
+        iyy="0.02188" iyz="0.0"
+        izz="0.0375"/>
     </inertial>
   </link>
@@ -56,9 +56,9 @@
     <inertial>
       <origin xyz="0.0 0.0 0.0" rpy="0 0 0"/>
-      <mass value="4.0"/>
+      <mass value="8.0"/>  <!-- Increased from 4.0 to concentrate weight at base -->
       <inertia
-          ixx="0.00443333"
-          iyy="0.00443333"
-          izz="0.0072"
+          ixx="0.00886666"
+          iyy="0.00886666"
+          izz="0.0144"
           ixy="0.0"
           iyz="0.0"
@@ -90,6 +90,6 @@
     <inertial>
       <origin xyz="0.0 -0.02561 0.00193" rpy="0 0 0"/>
-      <mass value="3.7"/>
-      <inertia ixx="0.010267" iyy="0.010267" izz="0.00666" ixy="0.0" iyz="0.0" ixz="0.0"/>
+      <mass value="4.5"/>  <!-- Increased from 3.7 to shift weight lower -->
+      <inertia ixx="0.012486" iyy="0.012486" izz="0.008100" ixy="0.0" iyz="0.0" ixz="0.0"/>
     </inertial>
     <visual>
@@ -117,6 +117,6 @@
     <inertial>
       <origin xyz="0.0 0.0 0.0" rpy="0 0 0"/>
-      <mass value="2.578"/>
-      <inertia ixx="0.006015" iyy="0.004988" izz="0.005608" ixy="0.0" iyz="0.0" ixz="0.0"/>
+      <mass value="1.0"/>  <!-- Reduced from 2.578 -->
+      <inertia ixx="0.002333" iyy="0.001935" izz="0.002175" ixy="0.0" iyz="0.0" ixz="0.0"/>
     </inertial>
     <visual>
@@ -144,6 +144,6 @@
     <inertial>
       <origin xyz="0.2125 0.0 0.11336" rpy="0 0 0"/>
-      <mass value="3.237"/>
-      <inertia ixx="0.084669" iyy="0.084669" izz="0.005827" ixy="0.0" iyz="0.0" ixz="0.0"/>
+      <mass value="1.0"/>  <!-- Reduced from 3.237 -->
+      <inertia ixx="0.026152" iyy="0.026152" izz="0.001800" ixy="0.0" iyz="0.0" ixz="0.0"/>
     </inertial>
     <visual>
@@ -170,6 +170,6 @@
     <inertial>
       <origin xyz="0.0 0.0 0.0" rpy="0 0 0"/>
-      <mass value="2.578"/>
-      <inertia ixx="0.006015" iyy="0.004988" izz="0.005608" ixy="0.0" iyz="0.0" ixz="0.0"/>
+      <mass value="0.5"/>  <!-- Reduced from 2.578 -->
+      <inertia ixx="0.001166" iyy="0.000968" izz="0.001088" ixy="0.0" iyz="0.0" ixz="0.0"/>
     </inertial>
     <visual>
@@ -196,6 +196,6 @@
     <inertial>
       <origin xyz="0.11993 0.0 0.0265" rpy="0 0 0"/>
-      <mass value="2.275"/>
-      <inertia ixx="0.004095" iyy="0.004095" izz="0.002049" ixy="0.0" iyz="0.0" ixz="0.0"/>
+      <mass value="0.5"/>  <!-- Reduced from 2.275 -->
+      <inertia ixx="0.000900" iyy="0.000900" izz="0.000450" ixy="0.0" iyz="0.0" ixz="0.0"/>
     </inertial>
     <visual>
@@ -223,6 +223,6 @@
     <inertial>
       <origin xyz="0.0 -0.0018 0.01634" rpy="0 0 0"/>
-      <mass value="1.219"/>
-      <inertia ixx="0.002110" iyy="0.002110" izz="0.002194" ixy="0.0" iyz="0.0" ixz="0.0"/>
+      <mass value="0.3"/>  <!-- Reduced from 1.219 -->
+      <inertia ixx="0.000519" iyy="0.000519" izz="0.000540" ixy="0.0" iyz="0.0" ixz="0.0"/>
     </inertial>
     <visual>
@@ -250,6 +250,6 @@
     <inertial>
       <origin xyz="0.0 0.0018 0.01634" rpy="0 0 0"/>
-      <mass value="1.219"/>
-      <inertia ixx="0.002110" iyy="0.002110" izz="0.002194" ixy="0.0" iyz="0.0" ixz="0.0"/>
+      <mass value="0.2"/>  <!-- Reduced from 1.219 -->
+      <inertia ixx="0.000346" iyy="0.000346" izz="0.000360" ixy="0.0" iyz="0.0" ixz="0.0"/>
     </inertial>
     <visual>
@@ -277,6 +277,6 @@
     <inertial>
       <origin xyz="0.0 0.001159 0.0" rpy="0 0 0"/>
-      <mass value="0.1879"/>
-      <inertia ixx="0.000132" iyy="0.000132" izz="0.000101" ixy="0.0" iyz="0.0" ixz="0.0"/>
+      <mass value="0.1"/>  <!-- Reduced from 0.1879 -->
+      <inertia ixx="0.000070" iyy="0.000070" izz="0.000054" ixy="0.0" iyz="0.0" ixz="0.0"/>
     </inertial>
     <visual>
